File: kicad/esp-p148-3way-crossover-retuned-quad-smd.kicad_pcb (KiCad board)
At the start: 4 copper layers, 149.6 x 63.5 mm, 90 parts, among them J1 TB-3P-3.5, J2 TB-2P-3.5, J3 TB-2P-3.5, J4 TB-2P-3.5, J5 TB-2P-3.5, Q1 MMBFJ112, Q2 MMBFJ112, Q3 MMBFJ112, SW1 DPDT LOCK, SW2 DPDT LOCK, SW3 DPDT LOCK, U1 MC33079, U2 MC33079, U3 MC33079

Commit message: Fix the KiCad exports: multi-unit parts, and J6 named after its own label
A routing tool reported U2, U3 "and loads of other components" missing on
import.  It was right, and there were two separate bugs.

1. MULTI-UNIT PARTS WERE EMITTED AS SEPARATE COMPONENTS.  The schematic
draws U1A..U1D and VR1A/VR1B; the board has one SOIC-14 called U1 and one
pot called VR1.  KiCad ties a symbol to a footprint by REFERENCE, so 17
schematic parts had no footprint and 6 footprints had no symbol.  They are
now proper multi-unit symbols: one lib_symbol per physical part with a
sub-symbol per unit, instances carrying (unit N) and the physical
reference, and a real crossover:<package> Footprint property.

The split cannot be guessed from the name - C3A/C3B look exactly like
U1A/U1B and are two real, separate capacitors - so unit_map() asks the
BOARD which designators physically exist.

2. J6 WAS NAMED LD1.  read_board() took the first silk text that looked
like a designator, and J6's footprint prints its pin labels LD1/LD2/LD3
before its own.  TEXT~P is the designator, TEXT~L is a plain label.  So
the seed carried a part that does not exist while the schematic's J6 had
no footprint.

Both files now agree exactly: 86 components each, no schematic part
without a footprint, no footprint without a symbol, U1-U3 as four-unit
symbols and VR1/VR2 as two-unit.

The schematic checker was extended rather than relaxed: it maps each
unit's pins back through the unit map, so this class of mismatch fails the
build instead of shipping.  It still rebuilds connectivity from the
emitted file's geometry alone - only the pin LABELS are translated from
section form (U1C.10) to physical form (U1.10).

Also: kicad/ was missing from check_all.py's GENERATED list, so changes
there were classed as source and never reported as drift.

Co-Authored-By: Claude Opus 5 <noreply@anthropic.com>
Claude-Session: https://claude.ai/code/session_01NEgWi6wEgHQCC2hjcx9DP1
Parts:
- removed LD1: MUTE, crossover:HDR-1X4
- added J6: MUTE, crossover:HDR-1X4, F.Cu at (188.2, 32.2)
Changed lines of the file:
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@@
  (at 188.163 32.224)
     (attr through_hole)
-    (property "Reference" "LD1" (at 0 0 0) (layer "F.SilkS") (effects (font (size 1 1) (thickness 0.15))))
+    (property "Reference" "J6" (at 0 0 0) (layer "F.SilkS") (effects (font (size 1 1) (thickness 0.15))))
     (property "Value" "MUTE" (at 0 0 0) (layer "F.Fab") (effects (font (size 1 1) (thickness 0.15))) (hide yes))
     (fp_line (start -1.397 5.08) (end -1.397 -5.08) (stroke (width 0.15) (type solid)) (layer "F.SilkS"))
