File: kicad/esp-p148-3way-crossover-retuned-quad-smd.kicad_sch (KiCad schematic)
At the start: 97 parts, among them J1 PWR, J2 IN, J3 HIGH, J4 MID, J5 LOW, J6 LEDS, Q1 MMBFJ112, Q2 MMBFJ112, Q3 MMBFJ112, SW1 DPDT LOCK, SW2 DPDT LOCK, SW3 DPDT LOCK, U1A MC33079, U1B MC33079, U1C MC33079, U1D MC33079, U2A MC33079, U2B MC33079, U2C MC33079, U2D MC33079, U3A MC33079, U3B MC33079, U3C MC33079, U3D MC33079

Commit message: Fix the KiCad exports: multi-unit parts, and J6 named after its own label
A routing tool reported U2, U3 "and loads of other components" missing on
import.  It was right, and there were two separate bugs.

1. MULTI-UNIT PARTS WERE EMITTED AS SEPARATE COMPONENTS.  The schematic
draws U1A..U1D and VR1A/VR1B; the board has one SOIC-14 called U1 and one
pot called VR1.  KiCad ties a symbol to a footprint by REFERENCE, so 17
schematic parts had no footprint and 6 footprints had no symbol.  They are
now proper multi-unit symbols: one lib_symbol per physical part with a
sub-symbol per unit, instances carrying (unit N) and the physical
reference, and a real crossover:<package> Footprint property.

The split cannot be guessed from the name - C3A/C3B look exactly like
U1A/U1B and are two real, separate capacitors - so unit_map() asks the
BOARD which designators physically exist.

2. J6 WAS NAMED LD1.  read_board() took the first silk text that looked
like a designator, and J6's footprint prints its pin labels LD1/LD2/LD3
before its own.  TEXT~P is the designator, TEXT~L is a plain label.  So
the seed carried a part that does not exist while the schematic's J6 had
no footprint.

Both files now agree exactly: 86 components each, no schematic part
without a footprint, no footprint without a symbol, U1-U3 as four-unit
symbols and VR1/VR2 as two-unit.

The schematic checker was extended rather than relaxed: it maps each
unit's pins back through the unit map, so this class of mismatch fails the
build instead of shipping.  It still rebuilds connectivity from the
emitted file's geometry alone - only the pin LABELS are translated from
section form (U1C.10) to physical form (U1.10).

Also: kicad/ was missing from check_all.py's GENERATED list, so changes
there were classed as source and never reported as drift.

Co-Authored-By: Claude Opus 5 <noreply@anthropic.com>
Claude-Session: https://claude.ai/code/session_01NEgWi6wEgHQCC2hjcx9DP1
Parts:
- U1: renamed from U1C; symbol crossover:U1C -> crossover:U1
- U1: renamed from U1D; symbol crossover:U1D -> crossover:U1
- U1: renamed from U1A; symbol crossover:U1A -> crossover:U1
- U1: renamed from U1B; symbol crossover:U1B -> crossover:U1
- U2: renamed from U2C; symbol crossover:U2C -> crossover:U2
- U2: renamed from U2B; symbol crossover:U2B -> crossover:U2
- U2: renamed from U2A; symbol crossover:U2A -> crossover:U2
- U2: renamed from U2D; symbol crossover:U2D -> crossover:U2
- U3: renamed from U3D; symbol crossover:U3D -> crossover:U3
- U3: renamed from U3C; symbol crossover:U3C -> crossover:U3
- U3: renamed from U3A; symbol crossover:U3A -> crossover:U3
- U3: renamed from U3B; symbol crossover:U3B -> crossover:U3
- VR1: renamed from VR1A; symbol crossover:VR1A -> crossover:VR1
- VR1: renamed from VR1B; symbol crossover:VR1B -> crossover:VR1
- VR2: renamed from VR2A; symbol crossover:VR2A -> crossover:VR2
- VR2: renamed from VR2B; symbol crossover:VR2B -> crossover:VR2
